Commit message: Added laser range setting

File: resources/models/pioneer3dx/defs/pioneer3dx_body.xacro (robot description, xacro)
@@ -273,5 +273,6 @@
                      min="${front_config['min_angle']}"
                      max="${front_config['max_angle']}"
-                     samples="${front_config['ray_count']}"/>
+                     samples="${front_config['ray_count']}"
+                     range="${front_config['range']}"/>
   </xacro:if>
   <!-- If enabled is set to true, add the laser. -->
@@ -285,5 +286,6 @@
                      min="${rear_config['min_angle']}"
                      max="${rear_config['max_angle']}"
-                     samples="${rear_config['ray_count']}"/>
+                     samples="${rear_config['ray_count']}"
+                     range="${front_config['range']}"/>
   </xacro:if>
   <!-- If enabled is set to true, add the kinect. -->

File: resources/models/pioneer3dx/defs/pioneer3dx_lasers.xacro (robot description, xacro)
@@ -2,5 +2,5 @@
 <robot xmlns:xacro="http://ros.org/wiki/xacro">
   <!-- Define a macro to add a laser sensor to the model based on given parameters. -->
-  <xacro:macro name="add_laser" params="descriptor visualize x y z yaw min max samples">
+  <xacro:macro name="add_laser" params="descriptor visualize x y z yaw min max samples range">
     <gazebo>
     <link name='hokuyo_${descriptor}_link'>
@@ -55,5 +55,5 @@
           <range>
             <min>0.08</min>
-            <max>10</max>
+            <max>${range}</max>
             <resolution>0.01</resolution>
           </range>

Commit message: Added navigation stack, fixed TF issues, new rviz config, new maps

File: resources/models/pioneer3dx/defs/pioneer3dx_body.xacro (robot description, xacro)
@@ -41,5 +41,5 @@
   	  <origin xyz="-0.045 0 0.148" rpy="0 0 0"/>
   	  <geometry name="pioneer_geom">
-    		<mesh filename="$(arg model_dir)/chassis.stl"/>
+    		<mesh filename="file://$(arg model_dir)/chassis.stl"/>
   	  </geometry>
   	  <material name="ChassisRed">
@@ -50,5 +50,5 @@
   	  <origin xyz="-0.045 0 0.148" rpy="0 0 0"/>
   	  <geometry>
-        <box size="0.4 0.28 0.17"/>
+        <box size="0.42 0.28 0.17"/>
         <!-- This is the correct bounding box, but x=0.43 crashes Gazebo? -->
     		<!--box size="0.43 0.28 0.17"/-->
@@ -69,5 +69,5 @@
   	  <origin xyz="0 0 0" rpy="0 0 0"/>
   	  <geometry name="pioneer_geom">
-    		<mesh filename="$(arg model_dir)/top.stl"/>
+    		<mesh filename="file://$(arg model_dir)/top.stl"/>
   	  </geometry>
   	  <material name="TopBlack">
@@ -85,5 +85,5 @@
   </joint>
   <!-- Swivel -->
-  <link name="swivel">
+  <link name="swivel_link">
   	<inertial>
   	  <mass value="0.1"/>
@@ -95,5 +95,5 @@
   	  <origin xyz="0 0 0" rpy="0 0 0"/>
   	  <geometry name="pioneer_geom">
-    		<mesh filename="$(arg model_dir)/swivel.stl"/>
+    		<mesh filename="file://$(arg model_dir)/swivel.stl"/>
   	  </geometry>
   	  <material name="swivel">
@@ -102,14 +102,14 @@
   	</visual>
   </link>
-  <gazebo reference="swivel">
+  <gazebo reference="swivel_link">
   	<material value="Gazebo/Black"/>
   </gazebo>
   <joint name="base_swivel_joint" type="continuous">
   	<origin xyz="-0.185 0 0.055" rpy="0 0 0"/>
+  	<parent link="base_link"/>
+  	<child link="swivel_link"/>
   	<axis xyz="0 0 1"/>
     <limit effort="100" velocity="100" k_velocity="0" />
     <joint_properties damping="0.0" friction="0.0" />
-  	<parent link="base_link"/>
-  	<child link="swivel"/>
   </joint>
   <!-- Center Wheel + Hubcap -->
@@ -124,5 +124,5 @@
   	  <origin xyz="0 0 0" rpy="0 0 0"/>
   	  <geometry name="pioneer_geom">
-    		<mesh filename="$(arg model_dir)/center_hubcap.stl"/>
+    		<mesh filename="file://$(arg model_dir)/center_hubcap.stl"/>
   	  </geometry>
   	  <material name="swivel">
@@ -136,10 +136,10 @@
   <joint name="swivel_hubcap_joint" type="continuous">
   	<origin xyz="-0.026 0 -0.016" rpy="0 0 0"/>
+  	<parent link="swivel_link"/>
+  	<child link="center_wheel"/>
   	<axis xyz="0 1 0"/>
   	<anchor xyz="0 0 0"/>
     <limit effort="100" velocity="100" k_velocity="0" />
     <joint_properties damping="0.0" friction="0.0" />
-  	<parent link="swivel"/>
-  	<child link="center_wheel"/>
   </joint>
   <link name="center_wheel">
@@ -153,5 +153,5 @@
   	  <origin xyz="0 0 0" rpy="0 0 0"/>
   	  <geometry name="pioneer_geom">
-    		<mesh filename="$(arg model_dir)/center_wheel.stl"/>
+    		<mesh filename="file://$(arg model_dir)/center_wheel.stl"/>
   	  </geometry>
   	  <material name="WheelBlack">
@@ -187,5 +187,5 @@
   	  <origin xyz="0 0 0" rpy="0 0 0"/>
   	  <geometry name="pioneer_geom">
-    		<mesh filename="$(arg model_dir)/front_sonar.stl"/>
+    		<mesh filename="file://$(arg model_dir)/front_sonar.stl"/>
   	  </geometry>
   	  <material name="SonarYellow">
@@ -212,5 +212,5 @@
   	  <origin xyz="0 0 0" rpy="0 0 0"/>
   	  <geometry name="pioneer_geom">
-    		<mesh filename="$(arg model_dir)/back_sonar.stl"/>
+    		<mesh filename="file://$(arg model_dir)/back_sonar.stl"/>
   	  </geometry>
   	  <material name="SonarYellow">
@@ -245,7 +245,7 @@
       <robotBaseFrame>base_link</robotBaseFrame>
       <publishTf>1</publishTf>
-      <publishWheelTF>false</publishWheelTF>
+      <publishWheelTF>true</publishWheelTF>
       <publishOdomTF>true</publishOdomTF>
-      <publishWheelJointState>false</publishWheelJointState>
+      <publishWheelJointState>true</publishWheelJointState>
       <rosDebugLevel>Warn</rosDebugLevel>
   	</plugin>
@@ -263,5 +263,5 @@
   	</plugin>
   </gazebo>
-  <!-- If enabled is set to true, add the laser. -->
+  <!-- If enabled is set to true, add the front laser. -->
   <xacro:if value="${front_laser == 1}">
     <xacro:add_laser descriptor="${front_config['descriptor']}"
@@ -276,5 +276,5 @@
                      range="${front_config['range']}"/>
   </xacro:if>
-  <!-- If enabled is set to true, add the laser. -->
+  <!-- If enabled is set to true, add the rear laser. -->
   <xacro:if value="${rear_laser == 1}">
     <xacro:add_laser descriptor="${rear_config['descriptor']}"
@@ -287,5 +287,5 @@
                      max="${rear_config['max_angle']}"
                      samples="${rear_config['ray_count']}"
-                     range="${front_config['range']}"/>
+                     range="${rear_config['range']}"/>
   </xacro:if>
   <!-- If enabled is set to true, add the kinect. -->

File: resources/models/pioneer3dx/defs/pioneer3dx_lasers.xacro (robot description, xacro)
@@ -3,40 +3,30 @@
   <!-- Define a macro to add a laser sensor to the model based on given parameters. -->
   <xacro:macro name="add_laser" params="descriptor visualize x y z yaw min max samples range">
-    <gazebo>
     <link name='hokuyo_${descriptor}_link'>
-      <pose frame=''>${x} ${y} ${z} 0 -0 ${yaw}</pose>
+      <!-- Not even slightly accurate -->
       <inertial>
-        <mass>0.1</mass>
-        <inertia>
-          <ixx>1</ixx>
-          <ixy>0</ixy>
-          <ixz>0</ixz>
-          <iyy>1</iyy>
-          <iyz>0</iyz>
-          <izz>1</izz>
-        </inertia>
-        <pose frame=''>0 0 0 0 -0 0</pose>
+        <origin xyz="0 0 -0.025" rpy="0 0 0"/>
+        <mass value="0.1"/>
+        <inertia
+          ixx="1.0" ixy="0.0" ixz="0.0"
+          iyy="1.0" iyz="0.0"
+          izz="1.0"/>
       </inertial>
-      <self_collide>0</self_collide>
-      <kinematic>0</kinematic>
-      <gravity>1</gravity>
-      <visual name='visual'>
+      <collision>
+        <origin xyz="0 0 -0.025" rpy="0 0 0"/>
         <geometry>
-          <mesh>
-            <!-- model_dir is an argument sent to the top level xml file (when setting robot_description) -->
-            <uri>file://$(arg model_dir)/hokuyo.dae</uri>
-          </mesh>
+          <box size="0.05 0.05 0.075"/>
         </geometry>
-        <material>
-          <shader type='pixel'>
-            <normal_map>__default__</normal_map>
-          </shader>
-        </material>
-        <pose frame=''>0 0 0 0 -0 0</pose>
-        <cast_shadows>1</cast_shadows>
-        <transparency>0</transparency>
+      </collision>
+      <visual>
+        <origin xyz="0 0 -0.025" rpy="0 0 0"/>
+        <geometry>
+          <mesh filename="file://$(arg model_dir)/hokuyo.dae" />
+        </geometry>
       </visual>
-      <sensor name='laser' type='ray'>
-        <pose frame=''>0.01 0 0.025 0 -0 0</pose>
+    </link>
+    <gazebo reference='hokuyo_${descriptor}_link'>
+      <sensor name='${descriptor}laser' type='ray'>
+        <pose frame=''>0 0 0 0 0 0</pose>
         <ray>
           <scan>
@@ -59,8 +49,8 @@
           </range>
         </ray>
-        <plugin name='laser' filename='libgazebo_ros_laser.so'>
+        <plugin name='${descriptor}laser' filename='libgazebo_ros_laser.so'>
           <!-- model_name is an argument sent to the top level xml file (when setting robot_description) -->
-          <topicName>/$(arg model_name)/${descriptor}scan</topicName>
-          <frameName>/${descriptor}scan_link</frameName>
+          <topicName>$(arg model_name)/${descriptor}scan</topicName>
+          <frameName>$(arg model_name)/hokuyo_${descriptor}_link</frameName>
         </plugin>
         <always_on>1</always_on>
@@ -68,134 +58,11 @@
         <visualize>${visualize}</visualize>
       </sensor>
-      <collision name='collision-base'>
-        <laser_retro>0</laser_retro>
-        <max_contacts>10</max_contacts>
-        <pose frame=''>0 0 -0.0145 0 -0 0</pose>
-        <geometry>
-          <box>
-            <size>0.05 0.05 0.041</size>
-          </box>
-        </geometry>
-        <surface>
-          <friction>
-            <ode>
-              <mu>1</mu>
-              <mu2>1</mu2>
-              <fdir1>0 0 0</fdir1>
-              <slip1>0</slip1>
-              <slip2>0</slip2>
-            </ode>
-            <torsional>
-              <coefficient>1</coefficient>
-              <patch_radius>0</patch_radius>
-              <surface_radius>0</surface_radius>
-              <use_patch_radius>1</use_patch_radius>
-              <ode>
-                <slip>0</slip>
-              </ode>
-            </torsional>
-          </friction>
-          <bounce>
-            <restitution_coefficient>0</restitution_coefficient>
-            <threshold>1e+06</threshold>
-          </bounce>
-          <contact>
-            <collide_without_contact>0</collide_without_contact>
-            <collide_without_contact_bitmask>1</collide_without_contact_bitmask>
-            <collide_bitmask>1</collide_bitmask>
-            <ode>
-              <soft_cfm>0</soft_cfm>
-              <soft_erp>0.2</soft_erp>
-              <kp>1e+13</kp>
-              <kd>1</kd>
-              <max_vel>0.01</max_vel>
-              <min_depth>0</min_depth>
-            </ode>
-            <bullet>
-              <split_impulse>1</split_impulse>
-              <split_impulse_penetration_threshold>-0.01</split_impulse_penetration_threshold>
-              <soft_cfm>0</soft_cfm>
-              <soft_erp>0.2</soft_erp>
-              <kp>1e+13</kp>
-              <kd>1</kd>
-            </bullet>
-          </contact>
-        </surface>
-      </collision>
-      <collision name='collision-top'>
-        <laser_retro>0</laser_retro>
-        <max_contacts>10</max_contacts>
-        <pose frame=''>0 0 0.0205 0 -0 0</pose>
-        <geometry>
-          <cylinder>
-            <radius>0.021</radius>
-            <length>0.029</length>
-          </cylinder>
-        </geometry>
-        <surface>
-          <friction>
-            <ode>
-              <mu>1</mu>
-              <mu2>1</mu2>
-              <fdir1>0 0 0</fdir1>
-              <slip1>0</slip1>
-              <slip2>0</slip2>
-            </ode>
-            <torsional>
-              <coefficient>1</coefficient>
-              <patch_radius>0</patch_radius>
-              <surface_radius>0</surface_radius>
-              <use_patch_radius>1</use_patch_radius>
-              <ode>
-                <slip>0</slip>
-              </ode>
-            </torsional>
-          </friction>
-          <bounce>
-            <restitution_coefficient>0</restitution_coefficient>
-            <threshold>1e+06</threshold>
-          </bounce>
-          <contact>
-            <collide_without_contact>0</collide_without_contact>
-            <collide_without_contact_bitmask>1</collide_without_contact_bitmask>
-            <collide_bitmask>1</collide_bitmask>
-            <ode>
-              <soft_cfm>0</soft_cfm>
-              <soft_erp>0.2</soft_erp>
-              <kp>1e+13</kp>
-              <kd>1</kd>
-              <max_vel>0.01</max_vel>
-              <min_depth>0</min_depth>
-            </ode>
-            <bullet>
-              <split_impulse>1</split_impulse>
-              <split_impulse_penetration_threshold>-0.01</split_impulse_penetration_threshold>
-              <soft_cfm>0</soft_cfm>
-              <soft_erp>0.2</soft_erp>
-              <kp>1e+13</kp>
-              <kd>1</kd>
-            </bullet>
-          </contact>
-        </surface>
-      </collision>
-    </link>
+    </gazebo>
+    <!-- Specify where the sensor link is in relation to base_link -->
     <joint name='base_${descriptor}_hokuyo' type='fixed'>
-      <parent>base_link</parent>
-      <child>hokuyo_${descriptor}_link</child>
-      <pose frame=''>0 0 0 0 -0 0</pose>
-      <physics>
-        <ode>
-          <limit>
-            <cfm>0</cfm>
-            <erp>0.2</erp>
-          </limit>
-          <suspension>
-            <cfm>0</cfm>
-            <erp>0.2</erp>
-          </suspension>
-        </ode>
-      </physics>
+      <origin xyz="${x} ${y} ${z}" rpy="0 0 ${yaw}" />
+      <parent link="base_link" />
+      <child link="hokuyo_${descriptor}_link" />
     </joint>
-    </gazebo>
   </xacro:macro>
 </robot>

File: resources/models/pioneer3dx/defs/pioneer3dx_wheel.xacro (robot description, xacro)
@@ -16,5 +16,5 @@
         <origin xyz="0 0 0" rpy="0 0 0"/>
         <geometry name="pioneer_geom">
-          <mesh filename="$(arg model_dir)/${suffix}_wheel.stl"/>
+          <mesh filename="file://$(arg model_dir)/${suffix}_wheel.stl"/>
           <!-- <mesh filename="package://resources/models/pioneer3dx/meshes/${suffix}_wheel.stl"/> -->
         </geometry>
@@ -45,5 +45,5 @@
         <origin xyz="0 0 0" rpy="0 0 0"/>
         <geometry name="pioneer_geom">
-          <mesh filename="$(arg model_dir)/${suffix}_hubcap.stl"/>
+          <mesh filename="file://$(arg model_dir)/${suffix}_hubcap.stl"/>
         </geometry>
         <material name="HubcapYellow">
